File: ESP32_S3_DEVKIT_EL_V1_PCBWay Community/ESP32_S3_DEVKIT_EL_V1.kicad_sch (KiCad schematic)
At the start: 61 parts, among them J10 BUTTONS, J11 POTENCIOMETERS, J12 RJ31_Shielded, J3 LEDS, J7 Conn_01x06_Pin, J9 Conn_02x05_Odd_Even, U4 RA-02

Commit message: PlacaOtraVez
Parts:
- removed J12: RJ31_Shielded, Connector_RJ:RJ45_Amphenol_RJHSE5380, symbol Connector:RJ31_Shielded
Changed lines of the file:
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@@
-    )
-  )
-  (symbol (lib_id "Connector:RJ31_Shielded") (at 372.5 93.5 0) (unit 1)
-    (in_bom yes) (on_board yes) (dnp no) (fields_autoplaced)
-    (property "Reference" "J12" (at 372.5 76.2 0)
-      (effects (font (size 1.27 1.27)))
-    )
-    (property "Value" "RJ31_Shielded" (at 372.5 78.74 0)
-      (effects (font (size 1.27 1.27)))
-    )
-    (property "Footprint" "Connector_RJ:RJ45_Amphenol_RJHSE5380" (at 372.5 92.865 90)
-      (effects (font (size 1.27 1.27)) hide)
-    )
-    (property "Datasheet" "~" (at 372.5 92.865 90)
-      (effects (font (size 1.27 1.27)) hide)
-    )
-    (pin "6")
-    (pin "4")
-    (pin "5")
-    (pin "SH")
-    (pin "3")
-    (pin "8")
-    (pin "2")
-    (pin "7")
-    (pin "1")
-    (instances
-      (project "ESP32_S3_DEVKIT_EL_V1"
-        (path "/f69018d9-0152-4280-9f90-0ae50db24bb3"
-          (reference "J12") (unit 1)
-        )
-      )
     )
   )
