File: ESP32_S3_DEVKIT_EL_V1_PCBWay Community/ESP32_S3_DEVKIT_EL_V1.kicad_pcb (KiCad board)
At the start: 2 copper layers, 100 x 100.4 mm, 64 parts, among them J1 Conn_02x03_IDC, J10 BUTTONS, J11 POTENCIOMETERS, J12 RJ31_Shielded, J2 USB_B_Micro, J3 LEDS, J4 Conn_02x03_IDC, J5 Conn_02x03_IDC, J6 Screw_Terminal_01x02, J7 Conn_01x06_Pin, J8 USB_B_Micro, J9 Conn_02x05_Odd_Even, Q2 Q_NPN_BEC, Q3 Q_NPN_BEC, SW1 SW_Push, SW2 SW_Push, U1 CH340C, U2 ESP32-S3-WROOM-1, U3 3.3v 1A, U4 RA-02

Commit message: PlacaOtraVez
Parts:
- moved J7 81.9 mm to (48.4, 57.1)
Routing:
- net /RTS: track 30.5 -> 34.7 mm, vias 1 -> 2
- net /GPIO_20: track 74.3 -> 75.2 mm, vias 1 -> 2
- net /GPIO_19: track 73.5 -> 74.3 mm
- net /D-: track 14.1 -> 14.6 mm, vias 1 -> 2
- net Net-(Q2-B): track 15.1 -> 15.5 mm, vias 1 -> 2
- net /D+: vias 1 -> 2

Commit message: Ultima PCB
PCB Final
Parts:
- removed H1, H2: MountingHole_2.7mm_M2.5_DIN965_Pad, MountingHole:MountingHole_2.7mm_M2.5_DIN965_Pad
- removed RV4: 100K, Potentiometer_THT:Potentiometer_Bourns_3386P_Vertical
- added ?: , , F.Cu at (96.0, 3.90)
- added ?: , , F.Cu at (3.90, 96.2)
- added ?: , , F.Cu at (3.60, 4.00)
- added D1: Blue LED, LED_SMD:LED_1206_3216Metric, F.Cu at (45.0, 83.8)
- added G***: LOGO, Images:CentroSteamLogo, F.Cu at (11.0, 16.7)
- added G***: LOGO, Images:imagenMejora, F.Cu at (85.0, 96.4)
- added G***: LOGO, Images:imagenMejora, F.Cu at (96.0, 34.9)
- added J13: RJ25, Connector_RJ:RJ25_Wayconn_MJEA-660X1_Horizontal, F.Cu at (23.6, 10.0)
- added J14: RJ25, Connector_RJ:RJ25_Wayconn_MJEA-660X1_Horizontal, F.Cu at (10.2, 40.9)
- added J15: 12,15,17,18,19,20,21,22, Connector_PinHeader_2.54mm:PinHeader_1x08_P2.54mm_Vertical, F.Cu at (71.7, 35.8)
- added J16: ~, Connector_PinHeader_2.54mm:PinHeader_1x04_P2.54mm_Vertical, F.Cu at (45.8, 15.0)
- added J17: ~, Connector_PinHeader_2.54mm:PinHeader_1x04_P2.54mm_Vertical, F.Cu at (45.8, 18.9)
- added J18: ~, Connector_PinHeader_2.54mm:PinHeader_1x04_P2.54mm_Vertical, F.Cu at (30.6, 15.0)
- added J19: ~, Connector_PinHeader_2.54mm:PinHeader_1x04_P2.54mm_Vertical, F.Cu at (30.6, 18.9)
- added J20: ~, Connector_PinHeader_2.54mm:PinHeader_1x04_P2.54mm_Vertical, F.Cu at (15.3, 34.2)
- added J21: ~, Connector_PinHeader_2.54mm:PinHeader_1x04_P2.54mm_Vertical, F.Cu at (19.2, 34.2)
- added J22: GPIO, Connector_RJ:RJ25_Wayconn_MJEA-660X1_Horizontal, F.Cu at (10.2, 72.3)
- added J23: GPIO2, Connector_RJ:RJ25_Wayconn_MJEA-660X1_Horizontal, F.Cu at (10.2, 87.9)
- added J24: ~, Connector_PinHeader_2.54mm:PinHeader_1x04_P2.54mm_Vertical, F.Cu at (15.5, 50.1)
- added J25: ~, Connector_PinHeader_2.54mm:PinHeader_1x04_P2.54mm_Vertical, F.Cu at (19.3, 50.1)
- added J26: ~, Connector_PinHeader_2.54mm:PinHeader_1x04_P2.54mm_Vertical, F.Cu at (15.3, 66.3)
- added J27: ~, Connector_PinHeader_2.54mm:PinHeader_1x04_P2.54mm_Vertical, F.Cu at (19.1, 66.3)
- added J28: ~, Connector_PinHeader_2.54mm:PinHeader_1x04_P2.54mm_Vertical, F.Cu at (15.3, 81.0)
- added J29: ~, Connector_PinHeader_2.54mm:PinHeader_1x04_P2.54mm_Vertical, F.Cu at (19.0, 81.0)
- added J30: GND, Connector_PinHeader_2.54mm:PinHeader_1x08_P2.54mm_Vertical, F.Cu at (16.2, 92.8)
- added J31: 5v, Connector_PinHeader_2.54mm:PinHeader_1x08_P2.54mm_Vertical, F.Cu at (37.6, 96.5)
- added J32: Conn_01x03_Pin, Connector_PinHeader_2.54mm:PinHeader_1x03_P2.54mm_Vertical, F.Cu at (31.2, 75.5)
- added J33: GND, Connector_PinHeader_2.54mm:PinHeader_1x08_P2.54mm_Vertical, F.Cu at (37.6, 92.8)
- added R3: 330R, Resistor_SMD:R_1206_3216Metric, F.Cu at (45.0, 87.1)
- added SWITCH LORA: SLW-913535-2A-SMT, SWITCH SMD:SLW9135352ASMT, F.Cu at (53.3, 85.5)
- J1: value Conn_02x03_IDC -> 12,15,17,18,19,20,21,22; footprint Connector_IDC:IDC-Header_2x03_P2.54mm_Vertical -> Connector_PinHeader_2.54mm:PinHeader_1x08_P2.54mm_Vertical
- J11: value POTENCIOMETERS -> 5v; footprint Connector_PinHeader_2.54mm:PinHeader_1x04_P2.54mm_Vertical -> Connector_PinHeader_2.54mm:PinHeader_1x08_P2.54mm_Vertical
- J12: value RJ31_Shielded -> RJ25; footprint Connector_RJ:RJ45_Amphenol_RJHSE5380 -> Connector_RJ:RJ25_Wayconn_MJEA-660X1_Horizontal
- J4: value Conn_02x03_IDC -> 4,5,6,7,8,9,10,11; footprint Connector_IDC:IDC-Header_2x03_P2.54mm_Vertical -> Connector_PinHeader_2.54mm:PinHeader_1x08_P2.54mm_Vertical
- J5: value Conn_02x03_IDC -> 23,24,25,31; footprint Connector_IDC:IDC-Header_2x03_P2.54mm_Vertical -> Connector_PinHeader_2.54mm:PinHeader_1x04_P2.54mm_Vertical
- J7: value Conn_01x06_Pin -> 4,5,6,7,8,9,10,11; footprint Connector_PinHeader_2.54mm:PinHeader_1x06_P2.54mm_Vertical -> Connector_PinHeader_2.54mm:PinHeader_1x08_P2.54mm_Vertical
- J9: value Conn_02x05_Odd_Even -> ANSEL; footprint Connector_IDC:IDC-Header_2x05_P2.54mm_Vertical -> Connector_RJ:RJ25_Wayconn_MJEA-660X1_Horizontal
- LED 1: renamed from D7
- LED 2: renamed from D8
- LED 3: renamed from D9
- LED 4: renamed from D10
- moved J11 102.7 mm to (16.2, 96.5), turned to 90 degrees
- moved J5 88.0 mm to (94.3, 24.2), turned to 180 degrees
- moved J4 81.2 mm to (60.0, 8.20)
- moved J12 76.4 mm to (39.6, 10.0), turned to 180 degrees
- moved RV1 62.0 mm to (27.6, 70.1)
- moved RV2 61.8 mm to (38.5, 70.1)
- moved RV3 61.5 mm to (49.2, 70.2)
- moved J1 57.8 mm to (71.8, 31.8), turned to 90 degrees
- moved J7 51.3 mm to (63.9, 8.20)
- moved C5 29.7 mm to (23.1, 54.2)
- moved C6 29.7 mm to (30.8, 54.2)
- moved J10 29.7 mm to (30.8, 58.5)
- moved BT3 29.7 mm to (38.6, 47.7)
- moved BT1 29.7 mm to (23.5, 47.7)
- moved BT2 29.7 mm to (31.2, 47.7)
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- renumbered SW1 to BOOT, SW2 to RESET
Connections:
- J1 pad 1: /GPIO_18 -> /GPIO_08
- J1 pad 2: /GPIO_18 -> /GPIO_03
- J1 pad 3: /GPIO_17 -> /GPIO_09
- J1 pad 4: /GPIO_17 -> /GPIO_10
- J1 pad 5: GND -> /GPIO_11
- J1 pad 6: GND -> /GPIO_12
- J11 pad 1: /POT1 -> +3.3V
- J11 pad 2: /POT2 -> +3.3V
- J11 pad 3: /POT3 -> +3.3V
- J11 pad 4: /POT4 -> +3.3V
- J12 pad 1: unconnected-(J12-Pad1) -> +3.3V
- J12 pad 2: unconnected-(J12-Pad2) -> /GPIO_17
- J12 pad 3: unconnected-(J12-Pad3) -> /GPIO_17
- J12 pad 4: unconnected-(J12-Pad4) -> /GPIO_18
- J12 pad 5: unconnected-(J12-Pad5) -> /GPIO_18
- J12 pad 6: unconnected-(J12-Pad6) -> GND
- J4 pad 1: /GPIO_08 -> /GPIO_04
- J4 pad 2: /GPIO_08 -> /GPIO_05
- J4 pad 3: /GPIO_09 -> /GPIO_06
- J4 pad 4: /GPIO_09 -> /GPIO_07
- J4 pad 5: GND -> /GPIO_15
- J4 pad 6: GND -> /GPIO_16
- J5 pad 1: /GPIO_10 -> /GPIO_21
- J5 pad 2: /GPIO_12 -> /GPIO_47
- J5 pad 3: GND -> /GPIO_48
- J5 pad 4: /GPIO_13 -> /GPIO_38
- J7 pad 1: unconnected-(J7-Pin_1-Pad1) -> /GPIO_04
- J7 pad 2: unconnected-(J7-Pin_2-Pad2) -> /GPIO_05
- J7 pad 3: unconnected-(J7-Pin_3-Pad3) -> /GPIO_06
- J7 pad 4: unconnected-(J7-Pin_4-Pad4) -> /GPIO_07
- J7 pad 5: unconnected-(J7-Pin_5-Pad5) -> /GPIO_15
- J7 pad 6: unconnected-(J7-Pin_6-Pad6) -> /GPIO_16
- J9 pad 1: +5V -> +3.3V
- J9 pad 2: /GPIO_42_TMS -> /GPIO_04
- J9 pad 3: GND -> /GPIO_05
- J9 pad 4: /GPIO_39_TCK -> /GPIO_06
- J9 pad 5: GND -> /GPIO_07
- J9 pad 6: /GPIO_40_TDO -> GND
- U4 pad 1: Net-(U4-GND-Pad1) -> GND
- U4 pad 12: unconnected-(U4-SCK-Pad12) -> /GPIO_12
- U4 pad 13: unconnected-(U4-MISO-Pad13) -> /GPIO_13
- U4 pad 14: unconnected-(U4-MOSI-Pad14) -> /GPIO_11
- U4 pad 15: unconnected-(U4-NSS-Pad15) -> /GPIO_10
- U4 pad 16: Net-(U4-GND-Pad1) -> GND
- U4 pad 2: Net-(U4-GND-Pad1) -> GND
- U4 pad 3: unconnected-(U4-3.3V-Pad3) -> Net-(S1-NC_4)
- U4 pad 4: unconnected-(U4-RESET-Pad4) -> /GPIO_01
- U4 pad 5: unconnected-(U4-DI00-Pad5) -> /GPIO_02
- U4 pad 9: Net-(U4-GND-Pad1) -> GND
Routing:
- net +3.3V: track 126.7 -> 394.4 mm, vias 0 -> 3
- net /GPIO_12: track 0.00 -> 229.5 mm, vias 0 -> 1
- net /GPIO_10: track 0.00 -> 220.9 mm
- net /GPIO_13: track 0.00 -> 220.3 mm
- net /GPIO_11: track 0.00 -> 211.2 mm, vias 0 -> 2
- net /GPIO_48: track 0.00 -> 163.5 mm
- net /GPIO_47: track 0.00 -> 158.1 mm
- net /GPIO_38: track 0.00 -> 156.7 mm
- net /GPIO_09: track 0.00 -> 155.8 mm, vias 0 -> 3
- net /GPIO_21: track 0.00 -> 153.4 mm
- net /GPIO_14: track 0.00 -> 138.9 mm
- net /GPIO_05: track 0.00 -> 131.2 mm, vias 0 -> 2
- net /GPIO_03: track 0.00 -> 126.1 mm, vias 0 -> 3
- net /GPIO_16: track 0.00 -> 120.2 mm, vias 0 -> 2
- net /GPIO_01: track 0.00 -> 116.0 mm
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- added copper zone on B.Cu, net GND
- added copper zone on F.Cu, net GND
Other:
- board size 100 x 100.4 mm -> 100 x 100 mm
- board text added: "- +5v"
- board text added: "1"
- board text added: "3"
- board text added: "3V3"
- board text added: "4"
- board text added: "5V"
- board text added: "ANSEL"
- board text added: "CSO"
- board text added: "D10"
- board text added: "D11"
- board text added: "D12"
- board text added: "D13"
- board text added: "D14"
- board text added: "D15"
- board text added: "D16"
- board text added: "D17"
- board text added: "D18"
- board text added: "D21"
- board text added: "D3"
- board text added: "D38"
- board text added: "D4"
- board text added: "D47"
- board text added: "D48"
- board text added: "D5"
- board text added: "D6"
- board text added: "D7"
- board text added: "D8"
- board text added: "D9"
- board text added: "GND"
- board text added: "GPIO"
- board text added: "I2C"
- board text added: "LORA RA-02"
- board text added: "MISO"
- board text added: "MOSI"
- board text added: "RX"
- board text added: "SCK"
- board text added: "SCL"
- board text added: "SDA"
- board text added: "SPI"
- board text added: "TX"
- board text added: "UART"
- board text added: "USB OTG"
- board text added: "USB UART"

Commit message: Version de frabricacion 01
Routing:
- net +3.3V: track 394.4 -> 407.6 mm, vias 3 -> 4
- net GND: track 0.00 -> 3.95 mm, vias 8 -> 9
- net /GPIO_38: track 156.7 -> 154.7 mm
- net /GPIO_47: track 158.1 -> 156.2 mm
- net /GPIO_02: track 114.4 -> 115.9 mm
- net /GPIO_14: track 138.9 -> 137.6 mm
- net /GPIO_48: track 163.5 -> 162.5 mm
- net /U0TXD: track 62.2 -> 61.2 mm
- net /U0RXD: track 64.6 -> 63.6 mm
- net /BTN4: track 14.5 -> 13.5 mm
- net Net-(S1-NC_4): track 41.6 -> 40.6 mm
- net /GPIO_18: track 55.6 -> 56.5 mm
- net /GPIO_15: track 114.3 -> 115.0 mm
- net /LED3: track 6.81 -> 7.41 mm
- net /GPIO_09: track 155.8 -> 156.4 mm
